File: KiCad/Triggy.kicad_sch (KiCad schematic)
At the start: 14 parts, among them M1 Motor 3V, Q1 TIP41, SW1 Engage, SW2 Bypass

Commit message: Rename repo
Other:
- title: II86 -> Triggy
Changed lines of the file:
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@@
 	(paper "USLetter")
 	(title_block
-		(title "II86")
+		(title "Triggy")
 		(date "2025-04-17")
 		(rev "1")
@@
 		)
 		(instances
-			(project "II86"
+			(project "Triggy"
 				(path "/9e25e860-f065-4810-857f-e93d45f31fd5"
 					(reference "R2")
@@
 		)
 		(instances
-			(project "II86"
+			(project "Triggy"
 				(path "/9e25e860-f065-4810-857f-e93d45f31fd5"
 					(reference "R3")
@@
 		)
 		(instances
-			(project "II86"
+			(project "Triggy"
 				(path "/9e25e860-f065-4810-857f-e93d45f31fd5"
 					(reference "#PWR03")
@@
 		)
 		(instances
-			(project "II86"
+			(project "Triggy"
 				(path "/9e25e860-f065-4810-857f-e93d45f31fd5"
 					(reference "R5")
@@
 		)
 		(instances
-			(project "II86"
+			(project "Triggy"
 				(path "/9e25e860-f065-4810-857f-e93d45f31fd5"
 					(reference "SW2")
@@
 		)
 		(instances
-			(project "II86"
+			(project "Triggy"
 				(path "/9e25e860-f065-4810-857f-e93d45f31fd5"
 					(reference "D3")
@@
 		)
 		(instances
-			(project "II86"
+			(project "Triggy"
 				(path "/9e25e860-f065-4810-857f-e93d45f31fd5"
 					(reference "D2")
@@
 		)
 		(instances
-			(project "II86"
+			(project "Triggy"
 				(path "/9e25e860-f065-4810-857f-e93d45f31fd5"
 					(reference "R4")
